Commit message: playing with stl format

File: galileo_ramp/track/track.urdf (robot description, URDF)
Before this commit: robot track.urdf, 1 links, 0 joints
Links:
- link baseLink: geometry collision mesh filename=track.obj scale=1. 1. 1.; visual mesh filename=track.stl scale=1. 1. 1.

Commit message: track physics appears to work

File: galileo_ramp/track/track.urdf (robot description, URDF)
Before this commit: robot track.urdf, 1 links, 0 joints
Links:
- link baseLink: geometry collision mesh filename=track.stl scale=1. 1. 1.; visual mesh filename=track.stl scale=1. 1. 1.
